Commit message: Add files via upload

File: rslk_ws/src/rslk/urdf/rslk.xacro (robot description, xacro)
@@ -15,5 +15,5 @@
       <origin xyz="0 0 -0.02" rpy=" 0 0 0"/>
       <geometry>
-        <cylinder length="0.020" radius="0.166"/>
+        <cylinder length="0.010" radius="0.0815"/>
       </geometry>
     </collision>
@@ -21,41 +21,53 @@
       <origin xyz="0 0 -0.02" rpy=" 0 0 0"/>
       <geometry>
-       <cylinder length="0.021" radius="0.167"/>
+       <cylinder length="0.011" radius="0.0815"/>
       </geometry>
     </visual>
     <collision name='back_caster_collision'>
-      <origin xyz="-0.1 0 -0.04" rpy=" 0 0 0"/>
+      <origin xyz="-0.062 0 -0.026" rpy=" 0 0 0"/>
       <geometry>
-        <sphere radius="0.0299"/>
+        <sphere radius="0.0114"/>
       </geometry>
     </collision>
     <visual name='back_caster_visual'>
-      <origin xyz="-0.1 0 -0.04" rpy=" 0 0 0"/>
+      <origin xyz="-0.062 0 -0.026" rpy=" 0 0 0"/>
       <geometry>
-        <sphere radius="0.03"/>
+        <sphere radius="0.0115"/>
       </geometry>
     </visual>
     <collision name='right_wheel_collision'>
-      <origin xyz="0 0.063 0" rpy=" 0 1.5707 1.5707"/>
+      <origin xyz="0 0.074 0" rpy=" 0 1.5707 1.5707"/>
       <geometry>
-        <cylinder length="0.00799" radius="0.0699"/>
+        <cylinder length="0.00799" radius="0.0349"/>
       </geometry>
     </collision>
     <visual name='right_wheel_visual'>
-      <origin xyz="0.0 0.064 0.0" rpy="0 1.5707 1.5707"/>
+      <origin xyz="0.0 0.074 0.0" rpy="0 1.5707 1.5707"/>
       <geometry>
-       <cylinder length="0.008" radius="0.07"/>
+       <cylinder length="0.008" radius="0.035"/>
+      </geometry>
+    </visual>
+    <collision name='motor_board_collision'>
+      <origin xyz="0 0.0 0" rpy=" 0 0 0"/>
+      <geometry>
+        <box size="0.112 0.1 0.002"/>
+      </geometry>
+    </collision>
+    <visual name='motor_board_visual'>
+      <origin xyz="0.0 0.0 0.0" rpy="0 0 0"/>
+      <geometry>
+        <box size="0.112 0.1 0.002"/>
       </geometry>
     </visual>
     <collision name='left_wheel_collision'>
-      <origin xyz="0 -0.063 0" rpy=" 0 1.5707 1.5707"/>
+      <origin xyz="0 -0.074 0" rpy=" 0 1.5707 1.5707"/>
       <geometry>
-        <cylinder length="0.00799" radius="0.0699"/>
+        <cylinder length="0.00799" radius="0.0349"/>
       </geometry>
     </collision>
     <visual name='left_wheel_visual'>
-      <origin xyz="0.0 -0.064 0.0" rpy="0 1.5707 1.5707"/>
+      <origin xyz="0.0 -0.074 0.0" rpy="0 1.5707 1.5707"/>
       <geometry>
-       <cylinder length="0.008" radius="0.07"/>
+       <cylinder length="0.008" radius="0.035"/>
       </geometry>
     </visual>
